File: Kicad/JR-200_SD.kicad_pcb (KiCad board)
At the start: 2 copper layers, 100 x 100 mm, 27 parts, among them J1 Conn_02x25_Odd_Even, J2 Micro_SD_Card_Kit, J3 MicroSD Card Adapter, U1 74LS04, U2 74LS30, U3 74LS04, U4 74LS30, U5 27512, U6 74LS00, U7 74LS30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

Commit message: Add files via upload
Parts:
- U6: value 74LS00 -> 74LS04
- U8: value 8255 -> 6821
- moved C4 3.14 mm to (132.1, 96.5), turned to 180 degrees
- moved U8 0.35 mm to (138.1, 148.6)
Connections:
- J1 pad 44: (no net) -> /~VMA
- U6 pad 10: Net-(U1-Pad8) -> Net-(U6-Pad10)
- U6 pad 11: Net-(U6-Pad11) -> /CLOCK
- U6 pad 12: /~RESET -> (no net)
- U6 pad 13: /~RESET -> GND
- U6 pad 2: /A3 -> Net-(U6-Pad2)
- U6 pad 3: Net-(U6-Pad3) -> /A2
- U6 pad 4: /A2 -> Net-(U6-Pad4)
- U6 pad 5: /A2 -> /~VMA
- U7 pad 11: Net-(U6-Pad6) -> Net-(U6-Pad4)
- U7 pad 6: Net-(U6-Pad3) -> Net-(U6-Pad2)
- U8 pad 1: Net-(U8-Pad1) -> GND
- U8 pad 11: (no net) -> Net-(U8-Pad11)
- U8 pad 12: (no net) -> Net-(U8-Pad12)
- U8 pad 13: (no net) -> Net-(U8-Pad13)
- U8 pad 14: (no net) -> Net-(U8-Pad14)
- U8 pad 15: (no net) -> Net-(U8-Pad15)
- U8 pad 16: Net-(U8-Pad16) -> (no net)
- U8 pad 18: Net-(U8-Pad18) -> (no net)
- U8 pad 19: Net-(U8-Pad19) -> (no net)
- U8 pad 20: Net-(U8-Pad20) -> +5V
- U8 pad 21: Net-(U8-Pad21) -> Net-(U6-Pad8)
- U8 pad 22: Net-(U8-Pad22) -> Net-(U6-Pad6)
- U8 pad 23: Net-(U8-Pad23) -> Net-(U7-Pad8)
- U8 pad 24: Net-(U8-Pad24) -> Net-(U6-Pad6)
- U8 pad 25: Net-(U8-Pad25) -> Net-(U6-Pad10)
- U8 pad 26: +5V -> /DB7
- U8 pad 27: /DB7 -> /DB6
- U8 pad 28: /DB6 -> /DB5
- U8 pad 29: /DB5 -> /DB4
- U8 pad 30: /DB4 -> /DB3
- U8 pad 31: /DB3 -> /DB2
- U8 pad 32: /DB2 -> /DB1
- U8 pad 33: /DB1 -> /DB0
- U8 pad 34: /DB0 -> /~RESET
- U8 pad 35: Net-(U6-Pad11) -> /A1
- U8 pad 36: Net-(U6-Pad8) -> /A0
- U8 pad 5: /~RD -> Net-(U8-Pad5)
- U8 pad 6: Net-(U7-Pad8) -> Net-(U8-Pad6)
- U8 pad 7: GND -> Net-(U8-Pad7)
- U8 pad 8: /A1 -> Net-(U8-Pad8)
- U8 pad 9: /A0 -> Net-(U8-Pad9)
- U9 pad 10: Net-(U8-Pad23) -> Net-(U8-Pad7)
- U9 pad 11: Net-(U8-Pad24) -> Net-(U8-Pad8)
- U9 pad 12: Net-(U8-Pad25) -> Net-(U8-Pad9)
- U9 pad 17: Net-(U8-Pad10) -> Net-(U8-Pad14)
- U9 pad 18: Net-(U8-Pad16) -> Net-(U8-Pad15)
- U9 pad 19: Net-(U8-Pad4) -> Net-(U8-Pad10)
- U9 pad 20: Net-(U8-Pad3) -> Net-(U8-Pad11)
- U9 pad 5: Net-(U8-Pad18) -> Net-(U8-Pad2)
- U9 pad 6: Net-(U8-Pad19) -> Net-(U8-Pad3)
- U9 pad 7: Net-(U8-Pad20) -> Net-(U8-Pad4)
- U9 pad 8: Net-(U8-Pad21) -> Net-(U8-Pad5)
- U9 pad 9: Net-(U8-Pad22) -> Net-(U8-Pad6)
- U9 pad A4: Net-(U8-Pad2) -> Net-(U8-Pad12)
- U9 pad A5: Net-(U8-Pad1) -> Net-(U8-Pad13)
Routing:
- net Net-(U6-Pad11): track 77.0 -> 0.00 mm
- net Net-(U7-Pad8): track 138.2 -> 65.7 mm
- net /~VMA: track 0.00 -> 57.1 mm
- net Net-(U8-Pad16): track 56.0 -> 0.00 mm
- net Net-(U8-Pad20): track 55.4 -> 0.00 mm
- net Net-(U8-Pad13): track 0.00 -> 54.4 mm
- net Net-(U8-Pad15): track 0.00 -> 52.4 mm
- net Net-(U8-Pad11): track 0.00 -> 48.6 mm
- net Net-(U6-Pad10): track 0.00 -> 48.4 mm
- net Net-(U8-Pad21): track 48.0 -> 0.00 mm, vias 1 -> 0
- net Net-(U8-Pad12): track 0.00 -> 47.2 mm
- net Net-(U6-Pad2): track 0.00 -> 47.1 mm, vias 0 -> 1
- net Net-(U6-Pad8): track 89.2 -> 43.4 mm
- net Net-(U8-Pad14): track 0.00 -> 44.5 mm
- net Net-(U8-Pad22): track 44.4 -> 0.00 mm, vias 1 -> 0
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Other:
- board text added: "6821"
- board text added: "JR-200_SD Rev2.1"
- board text removed: "74LS00"
- board text removed: "8255"
- board text removed: "JR-200_SD Rev1.7"
